Commit message: add four wheels to urdf

File: src/innex_description/urdf/innex_1.urdf.xacro (robot description, xacro)
@@ -41,3 +41,35 @@
     </inertial>
   </link>
+    <xacro:macro name="wheel" params="name x y">
+    <joint name="${name}_wheel_joint" type="continuous">
+      <parent link="base_link"/>
+      <child link="${name}_wheel"/>
+      <origin xyz="${x * wheelbase / 2} ${y * track / 2} ${wheel_radius}"/>
+      <axis xyz="0 1 0"/>
+    </joint>
+    <link name="${name}_wheel">
+      <visual>
+        <origin rpy="${pi / 2} 0 0"/>
+        <geometry>
+          <cylinder radius="${wheel_radius}" length="${wheel_width}"/>
+        </geometry>
+      </visual>
+      <collision>
+        <origin rpy="${pi / 2} 0 0"/>
+        <geometry>
+          <cylinder radius="${wheel_radius}" length="${wheel_width}"/>
+        </geometry>
+      </collision>
+      <inertial>
+        <mass value="${wheel_mass}"/>
+        <inertia ixx="${wheel_mass * (3 * wheel_radius * wheel_radius + wheel_width * wheel_width) / 12}" ixy="0" ixz="0"
+                 iyy="${wheel_mass * wheel_radius * wheel_radius / 2}" iyz="0"
+                 izz="${wheel_mass * (3 * wheel_radius * wheel_radius + wheel_width * wheel_width) / 12}"/>
+      </inertial>
+    </link>
+  </xacro:macro>
+  <xacro:wheel name="front_left" x="1" y="1"/>
+  <xacro:wheel name="front_right" x="1" y="-1"/>
+  <xacro:wheel name="rear_left" x="-1" y="1"/>
+  <xacro:wheel name="rear_right" x="-1" y="-1"/>
 </robot>

Commit message: Colour the rover model

File: src/innex_description/urdf/innex_1.urdf.xacro (robot description, xacro)
@@ -14,4 +14,16 @@
   <xacro:property name="chassis_mass" value="56.0"/>
   <xacro:property name="wheel_mass" value="1.0"/>
+  <material name="carbon">
+    <color rgba="0.18 0.18 0.2 1"/>
+  </material>
+  <material name="tyre">
+    <color rgba="0.05 0.05 0.05 1"/>
+  </material>
+  <material name="hub">
+    <color rgba="0.7 0.7 0.72 1"/>
+  </material>
+  <material name="accent">
+    <color rgba="1.0 0.45 0.0 1"/>
+  </material>
   <xacro:macro name="box_inertia" params="mass x y z">
     <inertia ixx="${mass / 12 * (y * y + z * z)}" ixy="0" ixz="0"
@@ -26,8 +38,16 @@
   </joint>
   <link name="chassis">
-    <visual>
+    <visual name="body">
       <geometry>
         <box size="${chassis_length} ${chassis_width} ${chassis_height}"/>
       </geometry>
+      <material name="carbon"/>
+    </visual>
+    <visual name="front_plate">
+      <origin xyz="${chassis_length / 2 + 0.005} 0 0"/>
+      <geometry>
+        <box size="0.01 ${chassis_width - 0.04} 0.12"/>
+      </geometry>
+      <material name="accent"/>
     </visual>
     <collision>
@@ -49,9 +69,24 @@
     </joint>
     <link name="${name}_wheel">
-      <visual>
+      <visual name="tyre">
         <origin rpy="${pi / 2} 0 0"/>
         <geometry>
           <cylinder radius="${wheel_radius}" length="${wheel_width}"/>
         </geometry>
+        <material name="tyre"/>
+      </visual>
+      <visual name="hub">
+        <origin xyz="0 ${y * (wheel_width / 2 + 0.005)} 0" rpy="${pi / 2} 0 0"/>
+        <geometry>
+          <cylinder radius="0.09" length="0.01"/>
+        </geometry>
+        <material name="hub"/>
+      </visual>
+      <visual name="spoke">
+        <origin xyz="0 ${y * (wheel_width / 2 + 0.011)} 0"/>
+        <geometry>
+          <box size="0.17 0.012 0.03"/>
+        </geometry>
+        <material name="accent"/>
       </visual>
       <collision>

Commit message: Add front and rear OAK-D Pro cameras to the rover model and sim
## What and why

Adds the front and rear Luxonis OAK-D Pro camera sensors to the rover URDF and Gazebo Harmonic simulation.

Fixes INX-157

- Adds a reusable `oak_d_pro.xacro` macro with visual/collision geometry, physical inertials, and REP-103 optical frames (+Z forward, +X right, +Y down).
- Mounts front and rear cameras to the chassis in `innex_1.urdf.xacro`.
- Configures Gazebo Harmonic camera sensors with 640x400 resolution at 15 FPS and 1.2043 rad (69 deg) HFOV.
- Bridges camera image and camera_info topics to ROS 2 in `bridge.yaml` under `/oak_front/` and `/oak_rear/` matching depthai-ros conventions.

## Testing

- Verified with `colcon build --symlink-install` (0 warnings, 0 errors).
- Added `test_oak_d_pro_cameras` in `test_urdf.py` checking links, joints, parent-child tree, optical rotations, and Gazebo sensors.
- Added `test_front_camera_publishes` and `test_rear_camera_publishes` in `test_rover_sim.py` verifying active image publication and optical frame IDs in ROS 2.
- Full test suite passed: `colcon test` (34 tests, 0 failures).
- Measured simulation Real-Time Factor (RTF) in steady state: average RTF is 1.000 (exceeds >= 0.9 requirement).

File: src/innex_description/urdf/innex_1.urdf.xacro (robot description, xacro)
@@ -108,4 +108,12 @@
   <xacro:wheel name="rear_left" x="-1" y="1"/>
   <xacro:wheel name="rear_right" x="-1" y="-1"/>
+  <xacro:include filename="sensors/oak_d_pro.xacro"/>
+  <!-- Front and rear OAK-D Pro cameras -->
+  <xacro:oak_d_pro prefix="oak_front" parent="chassis">
+    <origin xyz="${chassis_length / 2 + 0.01 + 0.023 / 2} 0 0.05" rpy="0 0 0"/>
+  </xacro:oak_d_pro>
+  <xacro:oak_d_pro prefix="oak_rear" parent="chassis">
+    <origin xyz="${-chassis_length / 2 - 0.01 - 0.023 / 2} 0 0.05" rpy="0 0 ${pi}"/>
+  </xacro:oak_d_pro>
   <xacro:include filename="innex_1.gazebo.xacro"/>
 </robot>

Commit message: Add Ouster OS1-128 LiDAR to the rover model and sim
## What and why

Adds the Ouster OS1-128 LiDAR sensor to the rover URDF and Gazebo Harmonic simulation.

Fixes INX-158
Fixes INX-152

- Adds a reusable `ouster_os1.xacro` macro with cylindrical visual/collision geometry, physical inertials, and `os_sensor` / `os_lidar` frames matching `ouster-ros`.
- Mounts the LiDAR on the top-front of the chassis at 0.749 m total height, satisfying the 0.75 m height limit.
- Configures Gazebo Harmonic `gpu_lidar` sensor with 128 vertical channels (±21.2° VFOV) and 512 horizontal samples (360° HFOV) at 10 Hz.
- Bridges `/ouster/points` to ROS 2 in `bridge.yaml` as `sensor_msgs/msg/PointCloud2`.

## Testing

- Verified with `colcon build --symlink-install` (0 warnings, 0 errors).
- Added `test_ouster_os1_lidar` in `test_urdf.py` checking links, joints, parent-child hierarchy, and sensor parameters.
- Added `test_ouster_points_publishes` in `test_rover_sim.py` verifying active PointCloud2 publication on `/ouster/points` with `header.frame_id: os_sensor`.
- Full test suite passed: `colcon test` (36 tests, 0 failures).
- Measured simulation Real-Time Factor (RTF) in steady state with all sensors active (LiDAR + both cameras): average RTF is 1.000 (exceeds >= 0.9 requirement).

File: src/innex_description/urdf/innex_1.urdf.xacro (robot description, xacro)
@@ -116,4 +116,9 @@
     <origin xyz="${-chassis_length / 2 - 0.01 - 0.023 / 2} 0 0.05" rpy="0 0 ${pi}"/>
   </xacro:oak_d_pro>
+  <xacro:include filename="sensors/ouster_os1.xacro"/>
+  <!-- Ouster OS1-128 LiDAR mounted on front-top chassis -->
+  <xacro:ouster_os1 prefix="os_sensor" parent="chassis">
+    <origin xyz="0.20 0 ${chassis_height / 2 + 0.0583 / 2}" rpy="0 0 0"/>
+  </xacro:ouster_os1>
   <xacro:include filename="innex_1.gazebo.xacro"/>
 </robot>

Commit message: Add Ouster OS1-128 LiDAR to the rover model and sim
## What and why

Adds the Ouster OS1-128 LiDAR sensor to the rover URDF and Gazebo Harmonic simulation.

Fixes INX-158
Fixes INX-152

- Adds a reusable \ouster_os1.xacro\ macro with cylindrical visual/collision geometry, physical inertials, and \os_sensor\ / \os_lidar\ frames matching \ouster-ros\.
- Mounts the LiDAR on the top-front of the chassis at 0.749 m total height, satisfying the 0.75 m height limit.
- Configures Gazebo Harmonic \gpu_lidar\ sensor with 128 vertical channels (±21.2° VFOV) and 512 horizontal samples (360° HFOV) at 10 Hz.
- Bridges \/ouster/points\ to ROS 2 in \ridge.yaml\ as \sensor_msgs/msg/PointCloud2\.

## Testing

- Verified with \colcon build --symlink-install\ (0 warnings, 0 errors).
- Added \	est_ouster_os1_lidar\ in \	est_urdf.py\ checking links, joints, parent-child hierarchy, and sensor parameters.
- Added \	est_ouster_points_publishes\ in \	est_rover_sim.py\ verifying active PointCloud2 publication on \/ouster/points\ with \header.frame_id: os_sensor\.
- Full test suite passed: \colcon test\ (40 tests, 0 failures).
- Measured simulation Real-Time Factor (RTF) in steady state with all sensors active (LiDAR + both cameras): average RTF is 0.9998 (exceeds >= 0.9 requirement).
- Verified detection of 0.3 m rock (rock_7) 5.19 m in front of rover in Moon Yard simulation (64 return points on \/ouster/points\).

File: src/innex_description/urdf/innex_1.urdf.xacro (robot description, xacro)
@@ -118,4 +118,9 @@
     <origin xyz="${-chassis_length / 2 - 0.01 - 0.023 / 2} 0 0.05" rpy="0 0 ${pi}"/>
   </xacro:oak_d_pro>
+  <xacro:include filename="sensors/ouster_os1.xacro"/>
+  <!-- Ouster OS1-128 LiDAR mounted on front-top chassis -->
+  <xacro:ouster_os1 prefix="os_sensor" parent="chassis">
+    <origin xyz="0.20 0 ${chassis_height / 2 + 0.0583 / 2}" rpy="0 0 0"/>
+  </xacro:ouster_os1>
   <xacro:include filename="innex_1.gazebo.xacro"/>
 </robot>

Commit message: Add pitch parameter and 15 deg tilt to OAK cameras
Level camera mounts caused a 1.23 m near-ground blind spot and missed the arena AprilTag beacon when close to the rover.

- Adds a pitch parameter to the oak_d_pro macro defaulting to 0.0, using an intermediate mount frame so positive pitch rotates the camera downward regardless of mount heading.
- Configures a static 15 degree downward pitch in the rover URDF, reducing the blind spot to 0.67 m while keeping the arena beacon and horizon within the vertical field of view.
- Updates URDF tests to verify mount frames, pitch orientation, and optical frame transforms. All 34 tests pass in colcon test.

File: src/innex_description/urdf/innex_1.urdf.xacro (robot description, xacro)
@@ -109,9 +109,11 @@
   <xacro:wheel name="rear_right" x="-1" y="-1"/>
   <xacro:include filename="sensors/oak_d_pro.xacro"/>
+  <!-- Downward camera pitch (15 deg) covers near ground while keeping beacon in view -->
+  <xacro:property name="camera_pitch" value="${15 * pi / 180}"/>
   <!-- Front and rear OAK-D Pro cameras -->
-  <xacro:oak_d_pro prefix="oak_front" parent="chassis">
+  <xacro:oak_d_pro prefix="oak_front" parent="chassis" pitch="${camera_pitch}">
     <origin xyz="${chassis_length / 2 + 0.01 + 0.023 / 2} 0 0.05" rpy="0 0 0"/>
   </xacro:oak_d_pro>
-  <xacro:oak_d_pro prefix="oak_rear" parent="chassis">
+  <xacro:oak_d_pro prefix="oak_rear" parent="chassis" pitch="${camera_pitch}">
     <origin xyz="${-chassis_length / 2 - 0.01 - 0.023 / 2} 0 0.05" rpy="0 0 ${pi}"/>
   </xacro:oak_d_pro>

File: src/innex_description/urdf/sensors/oak_d_pro.xacro (robot description, xacro)
@@ -2,5 +2,5 @@
 <robot xmlns:xacro="http://www.ros.org/wiki/xacro" xmlns:gz="http://gazebosim.org/schema">
   <!-- Luxonis OAK-D Pro active stereo camera macro -->
-  <xacro:macro name="oak_d_pro" params="prefix parent *origin topic_prefix:='' horizontal_fov:=1.2043 width:=640 height:=400 rate:=15.0">
+  <xacro:macro name="oak_d_pro" params="prefix parent *origin pitch:=0.0 topic_prefix:='' horizontal_fov:=1.2043 width:=640 height:=400 rate:=15.0">
     <xacro:property name="camera_mass" value="0.091"/>
     <xacro:property name="camera_x" value="0.023"/>
@@ -8,9 +8,16 @@
     <xacro:property name="camera_z" value="0.030"/>
     <xacro:property name="actual_topic_prefix" value="${topic_prefix if topic_prefix else prefix}"/>
-    <!-- Mechanical / base mount joint and link -->
+    <!-- Mechanical mount joint and link -->
+    <joint name="${prefix}_mount_joint" type="fixed">
+      <parent link="${parent}"/>
+      <child link="${prefix}_mount_frame"/>
+      <xacro:insert_block name="origin"/>
+    </joint>
+    <link name="${prefix}_mount_frame"/>
+    <!-- Camera body joint tilted down by pitch parameter -->
     <joint name="${prefix}_joint" type="fixed">
-      <parent link="${parent}"/>
+      <parent link="${prefix}_mount_frame"/>
       <child link="${prefix}_frame"/>
-      <xacro:insert_block name="origin"/>
+      <origin xyz="0 0 0" rpy="0 ${pitch} 0"/>
     </joint>
     <link name="${prefix}_frame">

Commit message: Add front and rear OAK-D Pro cameras to the rover model and sim (#8)
Adds the front and rear Luxonis OAK-D Pro camera sensors to the rover URDF and Gazebo Harmonic simulation.

Fixes INX-157

- Adds a reusable oak_d_pro.xacro macro with visual/collision geometry, physical inertials, REP-103 optical frames, and a pitch parameter (default 0.0).
- Mounts front and rear cameras to the chassis in innex_1.urdf.xacro with a 15 degree downward pitch to cover near-ground obstacles and keep the arena AprilTag beacon in view.
- Configures Gazebo Harmonic camera sensors with 640x400 resolution at 15 FPS and 1.2043 rad (69 deg) HFOV.
- Bridges camera image and camera_info topics to ROS 2 in ridge.yaml under /oak_front/ and /oak_rear/ matching depthai-ros conventions.

## Testing

- Verified with colcon build --symlink-install (0 warnings, 0 errors).
- Added 	est_oak_d_pro_cameras in 	est_urdf.py checking mount frames, joints, parent-child tree, optical rotations, pitch angles, and Gazebo sensors.
- Added 	est_front_camera_publishes and 	est_rear_camera_publishes in 	est_rover_sim.py verifying active image publication and optical frame IDs in ROS 2.
- Full test suite passed: colcon test (34 tests, 0 failures).
- Measured simulation Real-Time Factor (RTF) in steady state: average RTF is 1.000 (exceeds >= 0.9 requirement).

File: src/innex_description/urdf/innex_1.urdf.xacro (robot description, xacro)
@@ -108,4 +108,14 @@
   <xacro:wheel name="rear_left" x="-1" y="1"/>
   <xacro:wheel name="rear_right" x="-1" y="-1"/>
+  <xacro:include filename="sensors/oak_d_pro.xacro"/>
+  <!-- Downward camera pitch (15 deg) covers near ground while keeping beacon in view -->
+  <xacro:property name="camera_pitch" value="${15 * pi / 180}"/>
+  <!-- Front and rear OAK-D Pro cameras -->
+  <xacro:oak_d_pro prefix="oak_front" parent="chassis" pitch="${camera_pitch}">
+    <origin xyz="${chassis_length / 2 + 0.01 + 0.023 / 2} 0 0.05" rpy="0 0 0"/>
+  </xacro:oak_d_pro>
+  <xacro:oak_d_pro prefix="oak_rear" parent="chassis" pitch="${camera_pitch}">
+    <origin xyz="${-chassis_length / 2 - 0.01 - 0.023 / 2} 0 0.05" rpy="0 0 ${pi}"/>
+  </xacro:oak_d_pro>
   <xacro:include filename="innex_1.gazebo.xacro"/>
 </robot>

Commit message: Fix LiDAR origin, remove os_lidar and update mount height
Align the Ouster OS1 coordinate frame with the hardware specification,
locating the link origin os_sensor at the bottom center of the housing.
Shift visual, collision, and inertial origins up by half-height, and mount
the sensor flush on the chassis top plate (z = chassis_height / 2).

Remove os_lidar link and joint from URDF since the ouster-ros driver
dynamically publishes this transform from sensor metadata on the physical
rover and sim topics use os_sensor.

Remove *.bat from .gitignore to keep PR changes scoped.

Refs INX-152

File: src/innex_description/urdf/innex_1.urdf.xacro (robot description, xacro)
@@ -121,5 +121,5 @@
   <!-- Ouster OS1-128 LiDAR mounted on front-top chassis -->
   <xacro:ouster_os1 prefix="os_sensor" parent="chassis">
-    <origin xyz="0.20 0 ${chassis_height / 2 + 0.0583 / 2}" rpy="0 0 0"/>
+    <origin xyz="0.20 0 ${chassis_height / 2}" rpy="0 0 0"/>
   </xacro:ouster_os1>
   <xacro:include filename="innex_1.gazebo.xacro"/>

File: src/innex_description/urdf/sensors/ouster_os1.xacro (robot description, xacro)
@@ -14,4 +14,5 @@
     <link name="${prefix}">
       <visual>
+        <origin xyz="0 0 ${sensor_height / 2}" rpy="0 0 0"/>
         <geometry>
           <cylinder radius="${sensor_radius}" length="${sensor_height}"/>
@@ -20,4 +21,5 @@
       </visual>
       <collision>
+        <origin xyz="0 0 ${sensor_height / 2}" rpy="0 0 0"/>
         <geometry>
           <cylinder radius="${sensor_radius}" length="${sensor_height}"/>
@@ -25,4 +27,5 @@
       </collision>
       <inertial>
+        <origin xyz="0 0 ${sensor_height / 2}" rpy="0 0 0"/>
         <mass value="${sensor_mass}"/>
         <inertia ixx="${sensor_mass * (3 * sensor_radius * sensor_radius + sensor_height * sensor_height) / 12}" ixy="0" ixz="0"
@@ -31,11 +34,4 @@
       </inertial>
     </link>
-    <!-- Optical beam center frame (os_lidar) -->
-    <joint name="${prefix}_lidar_joint" type="fixed">
-      <parent link="${prefix}"/>
-      <child link="os_lidar"/>
-      <origin xyz="0 0 0.03618" rpy="0 0 0"/>
-    </joint>
-    <link name="os_lidar"/>
     <!-- Gazebo Harmonic GPU LiDAR Sensor -->
     <gazebo reference="${prefix}">
